File: 16Buttons_MCP23017.kicad_sch (KiCad schematic)
At the start: 27 parts, among them J3 Conn_01x07, U1 MCP23017_SP

Commit message: Updates.
Connections:
- no-connect marks 0 -> 16
Changed lines of the file:
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@@
   (junction (at 146.05 76.2) (diameter 0) (color 0 0 0 0)
   )
+  (no_connect (at 132.08 50.8))
+  (no_connect (at 146.05 50.8))
+  (no_connect (at 168.91 68.58))
+  (no_connect (at 189.23 86.36))
+  (no_connect (at 189.23 104.14))
+  (no_connect (at 189.23 68.58))
+  (no_connect (at 168.91 104.14))
+  (no_connect (at 168.91 86.36))
+  (no_connect (at 151.13 86.36))
+  (no_connect (at 151.13 68.58))
+  (no_connect (at 132.08 86.36))
+  (no_connect (at 132.08 104.14))
+  (no_connect (at 151.13 104.14))
+  (no_connect (at 132.08 68.58))
+  (no_connect (at 170.18 50.8))
+  (no_connect (at 184.15 50.8))
   (wire (pts (xy 137.16 52.07) (xy 137.16 157.48))
     (stroke (width 0) (type default) (color 0 0 0 0))
@@
     (stroke (width 0) (type default) (color 0 0 0 0))
   )
+  (wire (pts (xy 85.09 111.76) (xy 85.09 116.84))
+    (stroke (width 0) (type default) (color 0 0 0 0))
+  )
   (wire (pts (xy 163.83 104.14) (xy 163.83 152.4))
     (stroke (width 0) (type default) (color 0 0 0 0))
@@
   )
   (wire (pts (xy 132.08 58.42) (xy 146.05 58.42))
+    (stroke (width 0) (type default) (color 0 0 0 0))
+  )
+  (wire (pts (xy 85.09 172.72) (xy 85.09 177.8))
     (stroke (width 0) (type default) (color 0 0 0 0))
   )
@@
     )
   )
-  (symbol (lib_id "power:GND") (at 85.09 172.72 0) (unit 1)
+  (symbol (lib_id "power:GND") (at 85.09 177.8 0) (unit 1)
     (in_bom yes) (on_board yes) (fields_autoplaced)
-    (property "Reference" "#PWR0109" (id 0) (at 85.09 179.07 0)
-      (effects (font (size 1.27 1.27)) hide)
-    )
-    (property "Value" "GND" (id 1) (at 85.09 177.2825 0))
-    (property "Footprint" "" (id 2) (at 85.09 172.72 0)
-      (effects (font (size 1.27 1.27)) hide)
-    )
-    (property "Datasheet" "" (id 3) (at 85.09 172.72 0)
+    (property "Reference" "#PWR0109" (id 0) (at 85.09 184.15 0)
+      (effects (font (size 1.27 1.27)) hide)
+    )
+    (property "Value" "GND" (id 1) (at 85.09 182.3625 0))
+    (property "Footprint" "" (id 2) (at 85.09 177.8 0)
+      (effects (font (size 1.27 1.27)) hide)
+    )
+    (property "Datasheet" "" (id 3) (at 85.09 177.8 0)
       (effects (font (size 1.27 1.27)) hide)
     )
@@
     )
   )
-  (symbol (lib_id "power:+3.3V") (at 85.09 116.84 0) (unit 1)
+  (symbol (lib_id "power:+3.3V") (at 85.09 111.76 0) (unit 1)
     (in_bom yes) (on_board yes) (fields_autoplaced)
-    (property "Reference" "#PWR0110" (id 0) (at 85.09 120.65 0)
-      (effects (font (size 1.27 1.27)) hide)
-    )
-    (property "Value" "+3.3V" (id 1) (at 86.487 116.049 0)
+    (property "Reference" "#PWR0110" (id 0) (at 85.09 115.57 0)
+      (effects (font (size 1.27 1.27)) hide)
+    )
+    (property "Value" "+3.3V" (id 1) (at 86.487 110.969 0)
       (effects (font (size 1.27 1.27)) (justify left))
     )
-    (property "Footprint" "" (id 2) (at 85.09 116.84 0)
-      (effects (font (size 1.27 1.27)) hide)
-    )
-    (property "Datasheet" "" (id 3) (at 85.09 116.84 0)
-      (effects (font (size 1.27 1.27)) hide)
-    )
+    (property "Footprint" "" (id 2) (at 85.09 111.76 0)
+      (effects (font (size 1.27 1.27)) hide)
+    )
+    (property "Datasheet" "" (id 3) (at 85.09 111.76 0)
+      (effects (font (size 1.27 1.27)) hide)
+    )
