File: 16Buttons_MCP23017.kicad_pcb (KiCad board)
At the start: 2 copper layers, 52.8 x 68.6 mm, 27 parts, among them J3 Conn_01x07, U1 MCP23017_SP

Commit message: Updates.
Other:
- board text added: "Gnd"
- board text added: "IntA"
- board text added: "IntB"
- board text added: "Rst"
- board text added: "SCL"
- board text added: "SDA"
- board text added: "Vcc"
Changed lines of the file:
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@@
     (autoplace_cost90 3)
     (attr through_hole)
-    (fp_text reference "J3" (at 2.54 -5.085 180) (layer "B.SilkS")
+    (fp_text reference "J3" (at -0.254 2.535 -90) (layer "B.SilkS")
       (effects (font (size 1 1) (thickness 0.15)) (justify mirror))
     )
@@
   (gr_line (start 133.096 91.44) (end 133.096 93.98) (layer "Edge.Cuts") (width 0.1))
   (gr_arc (start 129.54 109.728) (mid 128.103159 109.132841) (end 127.508 107.696) (layer "Edge.Cuts") (width 0.1))
-  (gr_text "-" (at 124.714 132.08) (layer "B.Mask")
+  (gr_text "Rst" (at 106.68 131.064) (layer "B.SilkS")
+    (effects (font (size 1 1) (thickness 0.15)) (justify mirror))
+  )
+  (gr_text "-" (at 124.714 132.08) (layer "B.SilkS")
     (effects (font (size 2 2) (thickness 0.3)) (justify mirror))
   )
-  (gr_text "+" (at 124.714 127) (layer "B.Mask")
+  (gr_text "IntA" (at 101.6 131.064) (layer "B.SilkS")
+    (effects (font (size 1 1) (thickness 0.15)) (justify mirror))
+  )
+  (gr_text "Vcc" (at 96.52 131.064) (layer "B.SilkS")
+    (effects (font (size 1 1) (thickness 0.15)) (justify mirror))
+  )
+  (gr_text "+" (at 124.714 127) (layer "B.SilkS")
     (effects (font (size 3 3) (thickness 0.3)) (justify mirror))
   )
-  (gr_text "Kitecraft made this,\nand it's good enuff." (at 106.68 70.612) (layer "B.Mask")
+  (gr_text "Gnd" (at 99.06 132.588) (layer "B.SilkS")
+    (effects (font (size 1 1) (thickness 0.15)) (justify mirror))
+  )
+  (gr_text "SDA\n" (at 111.76 131.064) (layer "B.SilkS")
+    (effects (font (size 1 1) (thickness 0.15)) (justify mirror))
+  )
+  (gr_text "Kitecraft made this,\nand it's good enuff." (at 106.68 70.612) (layer "B.SilkS")
+    (effects (font (size 1 1) (thickness 0.15)) (justify mirror))
+  )
+  (gr_text "SCL" (at 109.22 132.588) (layer "B.SilkS")
+    (effects (font (size 1 1) (thickness 0.15)) (justify mirror))
+  )
+  (gr_text "IntB" (at 104.14 132.588) (layer "B.SilkS")
     (effects (font (size 1 1) (thickness 0.15)) (justify mirror))
   )
@@
   (arc (start 107.95 124.045786) (mid 107.87388 124.428469) (end 107.657107 124.752893) (width 0.25) (layer "F.Cu") (net 1))
   (segment (start 94.742 85.416) (end 98.402 85.416) (width 0.25) (layer "B.Cu") (net 2))
-  (segment (start 108.887933 125.046067) (end 108.937107 124.996893) (width 0.25) (layer "B.Cu") (net 21))
-  (segment (start 101.595 128.27) (end 103.080107 126.784893) (width 0.25) (layer "B.Cu") (net 21))
-  (segment (start 103.787214 126.492) (end 104.863069 126.492) (width 0.25) (layer "B.Cu") (net 21))
-  (segment (start 106.844536 125.33896) (end 108.180826 125.33896) (width 0.25) (layer "B.Cu") (net 21))
-  (segment (start 109.23 124.289786) (end 109.23 123.2) (width 0.25) (layer "B.Cu") (net 21))
-  (segment (start 105.570175 126.199107) (end 106.13743 125.631853) (width 0.25) (layer "B.Cu") (net 21))
-  (arc (start 104.863069 126.492) (mid 105.245752 126.41588) (end 105.570175 126.199107) (width 0.25) (layer "B.Cu") (net 21))
-  (arc (start 103.080107 126.784893) (mid 103.40453 126.56812) (end 103.787214 126.492) (width 0.25) (layer "B.Cu") (net 21))
-  (arc (start 108.937107 124.996893) (mid 109.15388 124.67247) (end 109.23 124.289786) (width 0.25) (layer "B.Cu") (net 21))
-  (arc (start 108.180826 125.33896) (mid 108.563509 125.26284) (end 108.887933 125.046067) (width 0.25) (layer "B.Cu") (net 21))
-  (arc (start 106.844536 125.33896) (mid 106.461853 125.41508) (end 106.13743 125.631853) (width 0.25) (layer "B.Cu") (net 21))
+  (segment (start 109.23 123.2) (end 109.23 124.201472) (width 0.25) (layer "B.Cu") (net 21))
+  (segment (start 109.054264 124.625736) (end 109.004893 124.675107) (width 0.25) (layer "B.Cu") (net 21))
+  (segment (start 108.297786 124.968) (end 105.311214 124.968) (width 0.25) (layer "B.Cu") (net 21))
+  (segment (start 104.604107 125.260893) (end 101.595 128.27) (width 0.25) (layer "B.Cu") (net 21))
+  (arc (start 109.23 124.201472) (mid 109.184328 124.431082) (end 109.054264 124.625736) (width 0.25) (layer "B.Cu") (net 21))
+  (arc (start 104.604107 125.260893) (mid 104.92853 125.04412) (end 105.311214 124.968) (width 0.25) (layer "B.Cu") (net 21))
+  (arc (start 109.004893 124.675107) (mid 108.68047 124.89188) (end 108.297786 124.968) (width 0.25) (layer "B.Cu") (net 21))
   (segment (start 116.85 116.161786) (end 116.85 115.58) (width 0.25) (layer "F.Cu") (net 22))
   (segment (start 109.215 128.27) (end 112.737107 124.747893) (width 0.25) (layer "F.Cu") (net 22))
@@
   (arc (start 111.477107 125.250893) (mid 111.69388 124.92647) (end 111.77 124.543786) (width 0.25) (layer "B.Cu") (net 24))
   (arc (start 110.525306 125.78848) (mid 110.907989 125.71236) (end 111.232413 125.495587) (width 0.25) (layer "B.Cu") (net 24))
-  (segment (start 113.068893 125.945107) (end 114.017107 124.996893) (width 0.25) (layer "B.Cu") (net 25))
-  (segment (start 106.675 128.27) (end 106.675 126.999528) (width 0.25) (layer "B.Cu") (net 25))
-  (segment (start 106.850736 126.575264) (end 106.895107 126.530893) (width 0.25) (layer "B.Cu") (net 25))
-  (segment (start 114.31 124.289786) (end 114.31 123.2) (width 0.25) (layer "B.Cu") (net 25))
-  (segment (start 107.602214 126.238) (end 112.361786 126.238) (width 0.25) (layer "B.Cu") (net 25))
-  (arc (start 106.895107 126.530893) (mid 107.21953 126.31412) (end 107.602214 126.238) (width 0.25) (layer "B.Cu") (net 25))
-  (arc (start 106.850736 126.575264) (mid 106.720672 126.769918) (end 106.675 126.999528) (width 0.25) (layer "B.Cu") (net 25))
-  (arc (start 113.068893 125.945107) (mid 112.74447 126.16188) (end 112.361786 126.238) (width 0.25) (layer "B.Cu") (net 25))
-  (arc (start 114.017107 124.996893) (mid 114.23388 124.67247) (end 114.31 124.289786) (width 0.25) (layer "B.Cu") (net 25))
+  (segment (start 107.436528 126.492) (end 111.947572 126.492) (width 0.25) (layer "B.Cu") (net 25))
+  (segment (start 106.675 128.27) (end 106.675 127.419214) (width 0.25) (layer "B.Cu") (net 25))
+  (segment (start 114.31 124.129572) (end 114.31 123.2) (width 0.25) (layer "B.Cu") (net 25))
+  (segment (start 106.967893 126.712107) (end 107.012264 126.667736) (width 0.25) (layer "B.Cu") (net 25))
+  (segment (start 112.654679 126.199107) (end 114.017107 124.836679) (width 0.25) (layer "B.Cu") (net 25))
+  (arc (start 106.967893 126.712107) (mid 106.75112 127.03653) (end 106.675 127.419214) (width 0.25) (layer "B.Cu") (net 25))
+  (arc (start 107.012264 126.667736) (mid 107.206918 126.537672) (end 107.436528 126.492) (width 0.25) (layer "B.Cu") (net 25))
+  (arc (start 114.31 124.129572) (mid 114.23388 124.512255) (end 114.017107 124.836679) (width 0.25) (layer "B.Cu") (net 25))
+  (arc (start 111.947572 126.492) (mid 112.330255 126.41588) (end 112.654679 126.199107) (width 0.25) (layer "B.Cu") (net 25))
   (segment (start 92.71 84.638214) (end 92.71 118.965786) (width 0.25) (layer "F.Cu") (net 26))
   (segment (start 92.417107 119.672893) (end 91.732893 120.357107) (width 0.25) (layer "F.Cu") (net 26))

Commit message: Adding Library
Routing:
- added copper zone on F.Cu, net GND
Other:
- board text added: "High"
- board text added: "Low"
- board text removed: "+"
- board text removed: "-"
Changed lines of the file:
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@@
     (effects (font (size 1 1) (thickness 0.15)) (justify mirror))
   )
-  (gr_text "-" (at 124.714 132.08) (layer "B.SilkS")
-    (effects (font (size 2 2) (thickness 0.3)) (justify mirror))
+  (gr_text "Low" (at 124.46 132.08 90) (layer "B.SilkS")
+    (effects (font (size 1 1) (thickness 0.15)) (justify mirror))
   )
   (gr_text "IntA" (at 101.6 131.064) (layer "B.SilkS")
@@
     (effects (font (size 1 1) (thickness 0.15)) (justify mirror))
   )
-  (gr_text "+" (at 124.714 127) (layer "B.SilkS")
-    (effects (font (size 3 3) (thickness 0.3)) (justify mirror))
+  (gr_text "High" (at 124.46 127 90) (layer "B.SilkS")
+    (effects (font (size 1 1) (thickness 0.15)) (justify mirror))
   )
   (gr_text "Gnd" (at 99.06 132.588) (layer "B.SilkS")
@@
   (arc (start 115.57 124.894214) (mid 115.64612 124.511531) (end 115.862893 124.187107) (width 0.25) (layer "B.Cu") (net 44))
   (arc (start 115.57 127.870786) (mid 115.64612 128.253469) (end 115.862893 128.577893) (width 0.25) (layer "B.Cu") (net 44))
+  (zone (net 2) (net_name "GND") (layer "F.Cu") (hatch edge 0.508)
+    (connect_pads yes (clearance 0.508))
+    (min_thickness 0.254) (filled_areas_thickness no)
+    (fill yes (thermal_gap 0.508) (thermal_bridge_width 0.508))
+    (polygon
+      (pts
+        (xy 127 133.985)
+        (xy 86.36 133.985)
+        (xy 86.36 66.675)
+        (xy 127 66.675)
+      )
+    )
+  )
   (zone (net 2) (net_name "GND") (layer "B.Cu") (hatch edge 0.508)
     (connect_pads yes (clearance 0.508))
