File: Hardware/16Buttons_MCP23017/16Buttons_MCP23017.kicad_pcb (KiCad board)
At the start: 2 copper layers, 52.8 x 68.6 mm, 27 parts, among them J3 Conn_01x07, U1 MCP23017_SP

Commit message: Everything seems to be built and working. PCB's and library both.
Parts:
- added C1: C, Capacitor_THT:C_Disc_D5.0mm_W2.5mm_P5.00mm, B.Cu at (93.1, 126.4)
Routing:
- added copper zone on F.Cu, net +3V3
- removed copper zone on F.Cu, net GND
