File: Hardware/16Buttons_MCP23017/16Buttons_MCP23017.kicad_sch (KiCad schematic)
At the start: 27 parts, among them J3 Conn_01x07, U1 MCP23017_SP

Commit message: Everything seems to be built and working. PCB's and library both.
Parts:
- added C1: C, Capacitor_THT:C_Disc_D5.0mm_W2.5mm_P5.00mm, symbol Device:C
Connections:
- net +3V3: now also C1.1
- net GND: now also C1.2
Changed lines of the file:
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@@
   (junction (at 132.08 93.98) (diameter 0) (color 0 0 0 0)
+  )
+  (junction (at 85.09 115.316) (diameter 0) (color 0 0 0 0)
   )
   (junction (at 151.13 76.2) (diameter 0) (color 0 0 0 0)
@@
     (stroke (width 0) (type default) (color 0 0 0 0))
   )
+  (wire (pts (xy 85.09 115.316) (xy 85.09 116.84))
+    (stroke (width 0) (type default) (color 0 0 0 0))
+  )
   (wire (pts (xy 102.87 160.02) (xy 139.7 160.02))
     (stroke (width 0) (type default) (color 0 0 0 0))
@@
     (stroke (width 0) (type default) (color 0 0 0 0))
   )
+  (wire (pts (xy 49.53 124.46) (xy 67.31 124.46))
+    (stroke (width 0) (type default) (color 0 0 0 0))
+  )
   (wire (pts (xy 151.13 93.98) (xy 158.75 93.98))
     (stroke (width 0) (type default) (color 0 0 0 0))
@@
     (stroke (width 0) (type default) (color 0 0 0 0))
   )
-  (wire (pts (xy 67.31 124.46) (xy 49.53 124.46))
-    (stroke (width 0) (type default) (color 0 0 0 0))
-  )
   (wire (pts (xy 184.15 139.7) (xy 102.87 139.7))
     (stroke (width 0) (type default) (color 0 0 0 0))
@@
     (stroke (width 0) (type default) (color 0 0 0 0))
   )
-  (wire (pts (xy 85.09 111.76) (xy 85.09 116.84))
+  (wire (pts (xy 85.09 111.76) (xy 85.09 115.316))
     (stroke (width 0) (type default) (color 0 0 0 0))
   )
@@
   )
   (wire (pts (xy 137.16 157.48) (xy 102.87 157.48))
+    (stroke (width 0) (type default) (color 0 0 0 0))
+  )
+  (wire (pts (xy 92.71 115.316) (xy 95.6564 115.316))
     (stroke (width 0) (type default) (color 0 0 0 0))
   )
@@
     (pin "4")
   )
+  (symbol (lib_id "Device:C") (at 88.9 115.316 90) (unit 1)
+    (in_bom yes) (on_board yes)
+    (property "Reference" "C1" (id 0) (at 91.44 114.2492 90))
+    (property "Value" "C" (id 1) (at 91.3892 116.4844 90))
+    (property "Footprint" "Capacitor_THT:C_Disc_D5.0mm_W2.5mm_P5.00mm" (id 2) (at 92.71 114.3508 0)
+      (effects (font (size 1.27 1.27)) hide)
+    )
+    (property "Datasheet" "~" (id 3) (at 88.9 115.316 0)
+      (effects (font (size 1.27 1.27)) hide)
+    )
+    (pin "1")
+    (pin "2")
+  )
   (symbol (lib_id "dk_Tactile-Switches:MJTP1230") (at 166.37 63.5 90) (unit 1)
     (in_bom yes) (on_board yes)
@@
     (pin "1")
   )
+  (symbol (lib_id "power:GND") (at 95.6564 115.316 90) (unit 1)
+    (in_bom yes) (on_board yes) (fields_autoplaced)
+    (property "Reference" "#PWR0112" (id 0) (at 102.0064 115.316 0)
+      (effects (font (size 1.27 1.27)) hide)
+    )
+    (property "Value" "GND" (id 1) (at 98.8314 115.7498 90)
+      (effects (font (size 1.27 1.27)) (justify right))
+    )
+    (property "Footprint" "" (id 2) (at 95.6564 115.316 0)
+      (effects (font (size 1.27 1.27)) hide)
+    )
+    (property "Datasheet" "" (id 3) (at 95.6564 115.316 0)
+      (effects (font (size 1.27 1.27)) hide)
+    )
+    (pin "1")
+  )
   (symbol (lib_id "dk_Tactile-Switches:MJTP1230") (at 148.59 99.06 90) (unit 1)
     (in_bom yes) (on_board yes)
@@
   )
   (symbol (lib_id "Interface_Expansion:MCP23017_SP") (at 85.09 144.78 0) (unit 1)
-    (in_bom yes) (on_board yes) (fields_autoplaced)
-    (property "Reference" "U1" (id 0) (at 87.1094 117.9535 0)
+    (in_bom yes) (on_board yes)
+    (property "Reference" "U1" (id 0) (at 79.5528 120.8532 0)
       (effects (font (size 1.27 1.27)) (justify left))
     )
@@
       (reference "#PWR0111") (unit 1) (value "GND") (footprint "")
     )
+    (path "/a25a2b2d-ed41-4dad-9481-5999a83606a5"
+      (reference "#PWR0112") (unit 1) (value "GND") (footprint "")
+    )
     (path "/be57f653-95b1-457c-a690-e64752bc4c21"
       (reference "A0") (unit 1) (value "Conn_01x03") (footprint "Connector_PinHeader_2.54mm:PinHeader_1x03_P2.54mm_Vertical")
@@
       (reference "A2") (unit 1) (value "Conn_01x03") (footprint "Connector_PinHeader_2.54mm:PinHeader_1x03_P2.54mm_Vertical")
     )
+    (path "/405e3491-1bb6-428b-81af-a8e410c94587"
+      (reference "C1") (unit 1) (value "C") (footprint "Capacitor_THT:C_Disc_D5.0mm_W2.5mm_P5.00mm")
+    )
     (path "/f42fc99a-e651-4f67-a40a-1ffa0ce6f622"
